File: N_CHANNEL/nChannel.sch (EAGLE design)
At the start: 26 parts

Commit message: Final PCB before testing
Parts:
- added C_VCC+, C_VCC-: 100u, rcl:C-US025-024X044
- RB_N: value 100k -> 10k
- RD2_P: value 40k -> 20k
- RMSR1_N, RMSR1_P, RMSR2_N, RMSR2_P: value 100k -> 2k
- RSHUNT_N, RSHUNT_P: value 52 -> 1
- renumbered R10 to RMSR4_P, R11 to RMSR1_P, R12 to RMSR3_P, R17 to RD2_P, R18 to RD1_P, R19 to RD1_N, R2 to RG3_P, R20 to RD2_N, R21 to RB_N, R22 to RMSR2_N, R23 to RSHUNT_N, R24 to RMSR4_N, R25 to RMSR1_N, R26 to RMSR3_N, R37 to RG2_P, R38 to RG4_P, R5 to RSHUNT_P, R9 to RMSR2_P
Connections:
- net N$34 renamed RVG_P
- removed net N$1: PIN-24.1, PIN-7.1, P_BUFF.D, RD1_N.1, RD1_P.1, RG4_P.1, RMSR4_N.2, RMSR4_P.2
- removed net N$30: RB_P.2
- removed net N$53: PIN-22.1, RG1_P.1
- new net 0: C_VCC+.2, C_VCC-.1, PIN-24.1, PIN-7.1, P_BUFF.D, RD1_N.1, RD1_P.1, RG4_P.1, RMSR4_N.2, RMSR4_P.2
- new net N$2: PIN-22.1, RB_P.2
- new net N$3: PIN-20.1, RG1_P.1
- net N$22: now also C_VCC-.2
- net N$32: now also C_VCC+.1
Other:
- note added: "ADC_N"
- note added: "ADC_P"
- note added: "DAC_D_N"
- note added: "DAC_G_N"
- note added: "Drain_N"
- note added: "Drain_P"
- note added: "GND"
- note added: "Gate_N"
- note added: "Gate_P"
- note added: "NC"
- note added: "Source_N"
- note added: "Source_P"
- note added: "VCC+"
- note added: "VCC-"
- note added: "VDAC_D_P"
- moved on the sheet: RG1_P
